File: hardware/bubblegum/bubblegum.sch (KiCad schematic (older format))
At the start: 148 parts, among them P1 RX_OUT, P10 CONN_1, P11 CONN_1, P12 CONN_1, P2 RX_ONLY, P3 SERIAL, P4 TX/RX, P5 CLK_IN, P6 TX_IN, P7 VCC, P8 SWITCH_CTRL, P9 CONN_1, T1 RX_IF_BALUN, T2 RX_BALUN, T3 RX_LO_BALUN2, T4 TX_BALUN, T5 RX_LO_BALUN1, T6 TX_IF_BALUN, T7 TX_LO_BALUN1, T8 TX_LO_BALUN2, U1 DMN2400, U10 TX_HIGHPASS_FILTER, U11 PE4140, U12 SKY13350, U13 TX_LOWPASS_FILTER, U14 DMC2400, U15 DMC2400, U16 GSG-74HC04, U17 SKY13350, U18 DMN2400, U19 NCP699, U2 SKY13350, U20 RX_LO_FILTER, U21 SKY13411, U22 SKY13411, U23 TX_LO_FILTER, U3 RX_HIGHPASS_FILTER, U4 SKY13350, U5 SKY13350, U6 PE4140, U7 RX_LOWPASS_FILTER, U8 SKY13350, U9 TRF3765

Commit message: hw
Parts:
- C1, C10, C11, C12, C13, C14, C15, C16, C17, C18, C19, C2, C20, C21, C22, C23, C24, C25, C26, C27, C28, C29, C3, C30, C31, C32, C33, C34, C35, C36, C37, C38, C39, C4, C40, C41, C42, C43, C44, C45, C46, C47, C48, C49, C5, C50, C51, C52, C53, C54, C55, C56, C57, C58, C59, C6, C60, C61, C62, C63, C64, C65, C66, C67, C68, C69, C7, C70, C71, C72, C73, C74, C75, C76, C77, C78, C79, C8, C80, C81, C82, C83, C84, C9: symbol C -> bubblegum-rescue:C
- D1, D2: symbol GSG-DIODE-TVS-BI -> hackrf:GSG-DIODE-TVS-BI
- FB1, FB2, FB3, FB4, FB5, FB6, FB7, FB8: symbol FILTER -> bubblegum-rescue:FILTER
- L3, L4, L5, L6: symbol INDUCTOR -> bubblegum-rescue:INDUCTOR
- P1, P2, P4, P6: symbol GSG-SMA-CONN -> hackrf:GSG-SMA-CONN
- P10, P11, P12, P9: symbol CONN_1 -> bubblegum-rescue:CONN_1
- P3, P8: symbol CONN_7X2 -> bubblegum-rescue:CONN_7X2
- P5: symbol CONN_2 -> bubblegum-rescue:CONN_2
- P7: symbol CONN_5X2 -> bubblegum-rescue:CONN_5X2
- R10, R13, R2, R3, R6, R7, R9: symbol R -> bubblegum-rescue:R
- T1, T6: symbol BALUN -> hackrf:BALUN
- T2, T3, T4, T5, T7, T8: symbol BALUN-B0310J50100AHF -> hackrf:BALUN-B0310J50100AHF
- U1, U14, U15, U18: symbol DMC2400 -> hackrf:DMC2400
- U10, U20, U23, U3: symbol FIL-DEA -> hackrf:FIL-DEA
- U11, U6: symbol PE4140 -> hackrf:PE4140
- U12, U17, U2, U4, U5, U8: symbol SKY13350 -> hackrf:SKY13350
- U13, U7: symbol FIL-LP0603 -> hackrf:FIL-LP0603
- U16: symbol GSG-74HC04 -> hackrf:GSG-74HC04
- U19: symbol NCP699 -> hackrf:NCP699
- U21, U22: symbol SKY13411 -> hackrf:SKY13411
- U9: symbol TRF3765 -> hackrf:TRF3765
Connections:
- wire segments 553 -> 678
