File: hardware/lemondrop/lemondrop.sch (KiCad schematic (older format))
At the start: 120 parts, among them P1 RX_SMA, P10 CONN_3, P11 1V8, P12 CONN_3, P13 CONN_3, P14 CONN_3, P15 CONN_3, P2 TX_SMA, P3 SPI, P4 VCC, P5 ADC/DAC, P6 XCVR_CTL, P7 CLOCK_CTL, P8 GSG-SMA-CONN, P9 CONN_2, T1 RX_BALUN, T2 TX_BALUN, U1 MAX5864, U2 MAX2837, U3 SI5351C, X1 GSG-XTAL4PIN

Commit message: hw
Parts:
- C1, C10, C11, C12, C13, C14, C15, C16, C17, C18, C19, C2, C20, C21, C22, C23, C24, C25, C26, C27, C28, C29, C3, C30, C31, C32, C33, C34, C35, C36, C37, C38, C39, C4, C40, C41, C42, C43, C44, C45, C46, C47, C48, C49, C5, C50, C51, C52, C53, C54, C6, C7, C8, C9: symbol C -> lemondrop-rescue:C
- L1, L2, L3, L4: symbol INDUCTOR -> lemondrop-rescue:INDUCTOR
- P1, P2, P8: symbol GSG-SMA-CONN -> hackrf:GSG-SMA-CONN
- P10, P12, P13, P14, P15: symbol CONN_3 -> lemondrop-rescue:CONN_3
- P11, P3, P4: symbol CONN_3X2 -> lemondrop-rescue:CONN_3X2
- P5: symbol CONN_20X2 -> lemondrop-rescue:CONN_20X2
- P6: symbol CONN_8X2 -> lemondrop-rescue:CONN_8X2
- P7: symbol CONN_6X2 -> lemondrop-rescue:CONN_6X2
- P9: symbol CONN_2 -> lemondrop-rescue:CONN_2
- R1, R10, R11, R12, R13, R14, R15, R16, R17, R18, R19, R2, R20, R21, R22, R23, R24, R25, R26, R27, R28, R29, R3, R30, R31, R32, R33, R34, R35, R36, R37, R38, R39, R4, R40, R41, R5, R6, R7, R8, R9: symbol R -> lemondrop-rescue:R
- T1, T2: symbol BALUN -> hackrf:BALUN
- U1: symbol MAX5864 -> hackrf:MAX5864
- U2: symbol MAX2837 -> hackrf:MAX2837
- U3: symbol SI5351C -> hackrf:SI5351C
- X1: symbol GSG-XTAL4PIN -> hackrf:GSG-XTAL4PIN
Connections:
- wire segments 377 -> 501
