File: hardware/licorice/licorice.sch (KiCad schematic (older format))
At the start: 113 parts, among them P1 TX-IN, P10 CONN_1, P11 CONN_1, P2 SERIAL, P3 RX-OUT, P4 ANTENNA, P5 CLK, P6 SWITCH_CTRL, P7 VCC, P8 CONN_1, P9 CONN_1, Q1 MOSFET_P, T1 MIX_IN_BALUN, T2 MIX_OUT_BALUN, U1 SKY13350, U10 SKY13350, U11 SKY13350, U12 SKY13317, U13 MGA-81563, U14 SKY13317, U15 GSG-74HC04, U16 GSG-74HC08, U2 SKY13350, U3 RX_LOWPASS_FILTER, U4 RFFC5072, U5 SKY13350, U6 SKY13350, U7 SKY13350, U8 RX_HIGHPASS_FILTER, U9 SKY13317

Commit message: hw
Parts:
- C1, C10, C11, C12, C13, C14, C15, C16, C17, C18, C19, C2, C20, C21, C22, C23, C24, C25, C26, C27, C28, C29, C3, C30, C31, C32, C33, C34, C35, C36, C37, C38, C39, C4, C40, C41, C42, C43, C44, C45, C46, C47, C48, C49, C5, C50, C51, C52, C53, C54, C55, C56, C57, C58, C59, C6, C60, C61, C62, C63, C64, C65, C66, C67, C68, C69, C7, C70, C8, C9: symbol C -> licorice-rescue:C
- D1: symbol GSG-DIODE-TVS-BI -> hackrf:GSG-DIODE-TVS-BI
- L1, L2, L3, L4, L5: symbol INDUCTOR -> licorice-rescue:INDUCTOR
- P1, P3, P4: symbol GSG-SMA-CONN -> hackrf:GSG-SMA-CONN
- P10, P11, P8, P9: symbol CONN_1 -> licorice-rescue:CONN_1
- P2: symbol CONN_5X2 -> licorice-rescue:CONN_5X2
- P5: symbol CONN_2 -> licorice-rescue:CONN_2
- P6, P7: symbol CONN_7X2 -> licorice-rescue:CONN_7X2
- Q1: symbol MOSFET_P -> licorice-rescue:MOSFET_P
- R1, R2, R3, R4, R5, R6, R7: symbol R -> licorice-rescue:R
- T1, T2: symbol BALUN-B0310J50100AHF -> hackrf:BALUN-B0310J50100AHF
- U1, U10, U11, U2, U5, U6, U7: symbol SKY13350 -> hackrf:SKY13350
- U12, U14, U9: symbol SKY13317 -> hackrf:SKY13317
- U13: symbol MGA-81563 -> hackrf:MGA-81563
- U15: symbol GSG-74HC04 -> hackrf:GSG-74HC04
- U16: symbol GSG-74HC08 -> hackrf:GSG-74HC08
- U3: symbol FIL-LP0603 -> hackrf:FIL-LP0603
- U4: symbol RFFC5072 -> hackrf:RFFC5072
- U8: symbol FIL-DEA -> hackrf:FIL-DEA
Connections:
- wire segments 378 -> 467
