File: hardware/lollipop/lollipop.sch (KiCad schematic (older format))
At the start: 130 parts, among them P1 TX-IN, P10 CONN_1, P11 CONN_1, P12 CONN_1, P2 TX/RX, P3 RX-only, P4 SERIAL, P5 RX-OUT, P6 CLK, P7 SWITCH_CTRL, P8 VCC, P9 CONN_1, T1 TX_IF_BALUN, T2 TX_BANDPASS_BALUN, T3 TX_LOWPASS_BALUN, T4 TX_HIGHPASS_BALUN, T5 RX_HIGHPASS_BALUN, T6 RX_LOWPASS_BALUN, T7 RX_BANDPASS_BALUN, T8 RX_IF_BALUN, U1 RFFC5071, U10 SKY13351, U11 TX_HIGHPASS_FILTER, U12 SKY13351, U13 RX_LOWPASS_FILTER, U14 SKY13351, U15 SKY13317, U16 SKY13351, U17 GSG-74HC04, U18 SKY13351, U19 GSG-74HC08, U2 SKY13351, U3 SKY13317, U4 SKY13351, U5 TX_LOWPASS_FILTER, U6 SKY13351, U7 SKY13351, U8 TX_HIGHPASS_FILTER, U9 SKY13351

Commit message: hw
Parts:
- C1, C10, C11, C12, C13, C14, C15, C16, C17, C18, C19, C2, C20, C21, C22, C23, C24, C25, C26, C27, C28, C29, C3, C30, C31, C32, C33, C34, C35, C36, C37, C38, C39, C4, C40, C41, C42, C43, C44, C45, C46, C47, C48, C49, C5, C50, C51, C52, C53, C54, C55, C56, C57, C58, C59, C6, C60, C61, C62, C63, C64, C65, C66, C67, C68, C69, C7, C70, C71, C72, C73, C74, C75, C76, C77, C8, C9: symbol C -> lollipop-rescue:C
- D1, D2: symbol GSG-DIODE-TVS-BI -> hackrf:GSG-DIODE-TVS-BI
- L1, L2, L3, L4, L5, L6: symbol INDUCTOR -> lollipop-rescue:INDUCTOR
- P1, P2, P3, P5: symbol GSG-SMA-CONN -> hackrf:GSG-SMA-CONN
- P10, P11, P12, P9: symbol CONN_1 -> lollipop-rescue:CONN_1
- P4: symbol CONN_5X2 -> lollipop-rescue:CONN_5X2
- P6: symbol CONN_2 -> lollipop-rescue:CONN_2
- P7: symbol CONN_7X2 -> lollipop-rescue:CONN_7X2
- P8: symbol CONN_3X2 -> lollipop-rescue:CONN_3X2
- R1, R2, R3, R4, R5, R6: symbol R -> lollipop-rescue:R
- T1, T2, T4, T5, T7, T8: symbol BALUN -> hackrf:BALUN
- T3, T6: symbol BALUN-RFXF9503 -> hackrf:BALUN-RFXF9503
- U1: symbol RFFC5071 -> hackrf:RFFC5071
- U10, U12, U14, U16, U18, U2, U4, U6, U7, U9: symbol SKY13351 -> hackrf:SKY13351
- U11, U8: symbol FIL-DEA -> hackrf:FIL-DEA
- U13, U5: symbol FIL-LP0603 -> hackrf:FIL-LP0603
- U15, U3: symbol SKY13317 -> hackrf:SKY13317
- U17: symbol GSG-74HC04 -> hackrf:GSG-74HC04
- U19: symbol GSG-74HC08 -> hackrf:GSG-74HC08
Connections:
- wire segments 439 -> 520
