File: hardware/neapolitan/baseband.sch (KiCad schematic (older format))
At the start: 77 parts, among them P14 XCVR_CLKOUT, P15 INTR, P18 OEB, P36 VAA, P39 SSP0_SCK, P40 SSP0_MOSI, P41 SSP0_MISO, P53 CS_XCVR, P55 TXENABLE, P56 RXENABLE, P57 XTAL2, P67 RSSI, P83 GND, P84 GND, P85 GND, P86 GND, P87 GND, P88 GND, P89 GND, P9 BASEBAND, P90 GND, P91 GND, P92 GND, Q3 MOSFET_P, T3 RX_BALUN, T4 TX_BALUN, U17 MAX2837, U19 SI5351C, X1 GSG-XTAL4PIN

Commit message: hw
Parts:
- C102, C104, C105, C106, C111, C112, C113, C114, C115, C116, C119, C120, C121, C122, C167, C169, C170, C80, C81, C84, C85, C86, C87, C88, C89, C90, C91, C92, C93, C94, C99: symbol C -> neapolitan-rescue:C
- FB2: symbol FILTER -> neapolitan-rescue:FILTER
- L14, L15, L16, L6, L7, L8, L9: symbol INDUCTOR -> neapolitan-rescue:INDUCTOR
- P14, P15, P18, P39, P40, P41, P53, P55, P56, P57, P67, P83, P84, P85, P86, P87, P88, P89, P90, P91, P92: symbol CONN_1 -> neapolitan-rescue:CONN_1
- P36: symbol CONN_2 -> neapolitan-rescue:CONN_2
- P9: symbol CONN_8X2 -> neapolitan-rescue:CONN_8X2
- Q3: symbol MOSFET_P -> neapolitan-rescue:MOSFET_P
- R104, R105, R11, R25, R26, R27, R28, R41, R85: symbol R -> neapolitan-rescue:R
- T3, T4: symbol BALUN -> hackrf:BALUN
- U17: symbol MAX2837 -> hackrf:MAX2837
- U19: symbol SI5351C -> hackrf:SI5351C
- X1: symbol GSG-XTAL4PIN -> hackrf:GSG-XTAL4PIN
Connections:
- wire segments 189 -> 244
