File: hardware/neapolitan/frontend.sch (KiCad schematic (older format))
At the start: 147 parts, among them J10 GND_CLIP, J2 RF-SHIELD-FRAME, J3 RF-SHIELD-COVER, J4 MOUNTING_HOLE, J5 MOUNTING_HOLE, J6 MOUNTING_HOLE, J7 MOUNTING_HOLE, J8 MOUNTING_HOLE, J9 MOUNTING_HOLE, P13 GPO1, P17 GPO6, P19 GPO3, P21 REF_IN, P27 MIXER_SDATA, P3 ANT_FAULT, P31 MIXER_SCLK, P32 MIXER_ENX, P33 MIXER_RESETX, P34 MIX_BYPASS, P35 !MIX_BYPASS, P4 ANTENNA, P42 TX, P43 RX, P44 HP, P45 LP, P46 TX_MIX_BP, P47 RX_MIX_BP, P48 TX_AMP, P49 RX_AMP, P50 AMP_BYPASS, P51 !TX_AMP_PWR, P52 !RX_AMP_PWR, P6 GPO4, P7 GPO2, Q1 MOSFET_P, Q2 MOSFET_P, T1 MIX_IN_BALUN, T2 MIX_OUT_BALUN, U1 SKY13350, U10 SKY13350, U11 SKY13350, U12 SKY13317, U13 MGA-81563, U14 SKY13317, U2 SKY13350, U20 AP2553W6-7, U25 MGA-81563, U3 RX_LOWPASS_FILTER, U4 RFFC5072, U5 SKY13350, U6 SKY13350, U7 SKY13350, U8 RX_HIGHPASS_FILTER, U9 SKY13317

Commit message: hw
Parts:
- C1, C10, C11, C12, C13, C14, C15, C16, C160, C161, C162, C163, C166, C17, C171, C18, C19, C2, C20, C21, C22, C23, C24, C25, C26, C27, C28, C29, C3, C30, C31, C32, C33, C34, C35, C36, C37, C38, C39, C4, C40, C41, C42, C43, C44, C45, C46, C47, C48, C49, C5, C50, C51, C52, C53, C54, C55, C56, C57, C58, C59, C6, C60, C61, C62, C63, C64, C65, C66, C67, C7, C70, C8, C9: symbol C -> neapolitan-rescue:C
- D1: symbol GSG-DIODE-TVS-BI -> hackrf:GSG-DIODE-TVS-BI
- J10, J4, J5, J6, J7, J8, J9, P13, P17, P19, P21, P27, P3, P31, P32, P33, P34, P35, P42, P43, P44, P45, P46, P47, P48, P49, P50, P51, P52, P6, P7: symbol CONN_1 -> neapolitan-rescue:CONN_1
- J2: symbol RF-SHIELD-FRAME -> hackrf:RF-SHIELD-FRAME
- J3: symbol RF-SHIELD-COVER -> hackrf:RF-SHIELD-COVER
- L1, L11, L12, L13, L2, L3, L4, L5: symbol INDUCTOR -> neapolitan-rescue:INDUCTOR
- P4: symbol GSG-RF-CONN -> hackrf:GSG-RF-CONN
- Q1, Q2: symbol MOSFET_P -> neapolitan-rescue:MOSFET_P
- R1, R2, R24, R29, R3, R33, R36, R4, R5, R6: symbol R -> neapolitan-rescue:R
- T1, T2: symbol BALUN-B0310J50100AHF -> hackrf:BALUN-B0310J50100AHF
- U1, U10, U11, U2, U5, U6, U7: symbol SKY13350 -> hackrf:SKY13350
- U12, U14, U9: symbol SKY13317 -> hackrf:SKY13317
- U13, U25: symbol MGA-81563 -> hackrf:MGA-81563
- U20: symbol NX5P2553GV -> gsg-symbols:NX5P2553GV
- U3: symbol FIL-LP0603 -> hackrf:FIL-LP0603
- U4: symbol RFFC5072 -> hackrf:RFFC5072
- U8: symbol FIL-DEA -> hackrf:FIL-DEA
Connections:
- wire segments 377 -> 448
