File: hardware/neapolitan/mcu.sch (KiCad schematic (older format))
At the start: 66 parts, among them J1 USB-MICRO-B, J11 BARREL_JACK, P1 !IO_INT, P2 !IO_RESET, P20 GPIO, P22 I2S, P28 SD, P5 LEDS, P80 SHIELD, Q5 MOSFET_P, Q6 MOSFET_P, Q7 MOSFET_P, U15 TCA6424A, U16 TCR2EF, U18 74LVC1G14, X2 FOX924B, X3 KT2520, X4 OH4

Commit message: hw
Parts:
- C155, C68, C69, C71, C72, C73, C74, C75, C76, C77, C78, C79, C82, C83, C95: symbol C -> neapolitan-rescue:C
- D10, D4, D8: symbol D_Schottky -> neapolitan-rescue:D_Schottky
- D2, D5, D6, D7: symbol LED -> neapolitan-rescue:LED
- FB1, FB3: symbol FILTER -> neapolitan-rescue:FILTER
- J1: symbol GSG-USB-MICRO-B-SHIELDED -> hackrf:GSG-USB-MICRO-B-SHIELDED
- J11: symbol BARREL_JACK -> neapolitan-rescue:BARREL_JACK
- L10: symbol INDUCTOR -> neapolitan-rescue:INDUCTOR
- P1, P2: symbol CONN_1 -> neapolitan-rescue:CONN_1
- P20, P28: symbol CONN_11X2 -> hackrf:CONN_11X2
- P22: symbol CONN_13X2 -> neapolitan-rescue:CONN_13X2
- P5: symbol CONN_3X2 -> neapolitan-rescue:CONN_3X2
- P80: symbol CONN_2 -> neapolitan-rescue:CONN_2
- Q5, Q6, Q7: symbol MOSFET_P -> neapolitan-rescue:MOSFET_P
- R10, R12, R13, R14, R15, R16, R17, R18, R19, R20, R21, R22, R23, R30, R31, R32, R35, R7, R73, R74, R75, R8, R9: symbol R -> neapolitan-rescue:R
- U15: symbol TCA6424A -> gsg-symbols:TCA6424A
- U16: symbol TCR2EF -> gsg-symbols:TCR2EF
- U18: symbol 74AHC1G14 -> neapolitan-rescue:74AHC1G14
- X2: symbol FOX924B -> gsg-symbols:FOX924B
- X3: symbol KT2520 -> gsg-symbols:KT2520
- X4: symbol OH4 -> gsg-symbols:OH4
Connections:
- wire segments 201 -> 243
