File: hardware/ice40board/ice40board/ice40board.sch (KiCad schematic (older format))
At the start: 8 parts, among them P1 Power, P2 Analog, P3 Digital, P4 Digital, P5 CONN_01X01, P6 CONN_01X01, P7 CONN_01X01, P8 CONN_01X01

Commit message: ice40 board
Parts:
- added C1, C2, C3, C4, C5, C6, C7, C8, C9: C, symbol Device:C
- added L1: L, symbol Device:L
- added R1, R2: R, symbol Device:R
- added U1: LTC3406ES5, Package_TO_SOT_SMD:TSOT-23-5, symbol Regulator_Switching:LTC3406ES5
- added U2: ICE40UP5K-SG48ITR, Package_DFN_QFN:QFN-48-1EP_7x7mm_P0.5mm_EP5.6x5.6mm, symbol FPGA_Lattice:ICE40UP5K-SG48ITR
Connections:
- net +3V3: now also C3.1, C4.1, C5.1, C6.1, U2.1 (VCCIO_2), U2.22 (SPI_VCCIO1), U2.24 (VPP_2V5), U2.33 (VCCIO_0)
- net GND: now also C3.2, C4.2, C5.2, C6.2, C7.2, C8.2, C9.2, U2.49 (GND)
- new net: C1.2, C2.2, R2.1, U1.2 (GND)
- new net: L1.2, U1.3 (SW)
- new net: C1.1, U1.4 (VIN)
- new net: R1.1, R2.2, U1.5 (VOUT)
- new net +1V2: C2.1, C7.1, C8.1, C9.1, L1.1, R1.2, U2.29 (VCCPLL), U2.30 (VCC), U2.5 (VCC)

Commit message: first gerber for ice40 board
Parts:
- added J2: Conn_01x04_Male, Connector_PinHeader_2.54mm:PinHeader_1x04_P2.54mm_Vertical, symbol Connector:Conn_01x04_Male
- added J3: Conn_01x08_Male, Connector_PinHeader_2.54mm:PinHeader_1x08_P2.54mm_Vertical, symbol Connector:Conn_01x08_Male
- C1: value C -> 4.7uF; footprint (none) -> Capacitor_SMD:C_1206_3216Metric
- C2: value C -> 10uF; footprint (none) -> Capacitor_SMD:C_1206_3216Metric
- C3: value C -> 0.1uF; footprint (none) -> Capacitor_SMD:C_0805_2012Metric
- C4, C5, C6, C7, C8, C9: footprint (none) -> Capacitor_SMD:C_0805_2012Metric
- L1: value L -> 2.2uH; footprint (none) -> Inductor_SMD:L_1210_3225Metric
- R1, R2: value R -> 100kohm; footprint (none) -> Resistor_SMD:R_1206_3216Metric
Connections:
- net +3V3: now also C1.1, U1.1 (RUN), U1.4 (VIN)
- net 0(Rx): now also U2.6 (IOB_13b)
- net 1(Tx): now also U2.9 (IOB_16a)
- net 10(**/SS): now also U2.16 (IOB_35b_SPI_SS)
- net 11(**/MOSI): now also U2.17 (IOB_33b_SPI_SI)
- net 12(MISO): now also U2.14 (IOB_32a_SPI_SO)
- net 13(SCK): now also U2.15 (IOB_34a_SPI_SCK)
- net 2: now also U2.10 (IOB_18a)
- net 3(**): now also U2.11 (IOB_20a)
- net 4: now also U2.12 (IOB_22b)
- net 6(**): now also U2.7 (CDONE)
- net 7: now also U2.8 (~CRESET)
- net A4(SDA): no longer P2.5 (Pin_5)
- net A5(SCL): no longer P2.6 (Pin_6)
- net GND: now also C1.2, C2.2, R2.1, U1.2 (GND)
- net at U2.39 (RGB0): now also J2.2 (Pin_2)
- net at U2.40 (RGB1): now also J2.3 (Pin_3)
- net at U2.41 (RGB2): now also J2.4 (Pin_4)
- net at U2.42 (IOT_51a): now also J2.1 (Pin_1)
- net at U2.2 (IOB_6a): now also J3.6 (Pin_6)
- net at U2.3 (IOB_9b): now also J3.8 (Pin_8)
- net at U2.4 (IOB_8a): now also J3.7 (Pin_7)
- net at U2.44 (IOB_3b_G6): now also J3.3 (Pin_3)
- net at U2.45 (IOB_5b): now also J3.5 (Pin_5)
- net at U2.46 (IOB_0a): now also J3.1 (Pin_1)
- net at U2.47 (IOB_2a): now also J3.2 (Pin_2)
- net at U2.48 (IOB_4a): now also J3.4 (Pin_4)
- no-connect marks 5 -> 39
Other:
- moved on the sheet: U2B
