File: hardware/ice40HX1Kboard/ice40HX1Kboard/ice40HX1Kboard/ice40HX1Kboard.sch (KiCad schematic (older format))
At the start: 30 parts

Commit message: ice40HX1K board: board without SRAM/ADC
Parts:
- added J1: Conn_02x05_Odd_Even, Connector_PinHeader_2.54mm:PinHeader_2x05_P2.54mm_Vertical, symbol Connector_Generic:Conn_02x05_Odd_Even
- added J2, J3, J4, J5: Conn_01x20_Male, Connector_PinHeader_2.54mm:PinHeader_1x20_P2.54mm_Vertical, symbol Connector:Conn_01x20_Male
- added J6: Conn_01x03_Male, Connector_PinHeader_2.54mm:PinHeader_1x03_P2.54mm_Vertical, symbol Connector:Conn_01x03_Male
- C1, C3: renamed from C?; footprint (none) -> Capacitor_SMD:C_1206_3216Metric
- C10, C11, C12, C13, C14, C15, C16, C17, C2, C4, C5, C6, C7, C8, C9: renamed from C?; value C -> 0.1uF; footprint (none) -> Capacitor_SMD:C_0805_2012Metric
- D1: renamed from D?; footprint (none) -> Capacitor_SMD:C_0603_1608Metric
- L1: renamed from L?; footprint (none) -> Inductor_SMD:L_1210_3225Metric
- R1, R2, R3, R4, R5, R6, R7, R8: renamed from R?; footprint (none) -> Resistor_SMD:R_1206_3216Metric
- U3: renamed from U?; footprint Package_QFP:LQFP-144_20x20mm_P0.5mm -> Package_QFP:LQFP-100_14x14mm_P0.5mm; symbol kilib:ICE40HX1K-VQ100(VQFP100) -> ice40HX1Kboard-rescue:ICE40HX1K-VQ100(VQFP100)-kilib
- gave numbers to parts that had none: 2
Connections:
- net IO1: now reaches U3.1 (IOL_1A)
- net IO1: now also J3.20 (Pin_20)
- net IO10: now reaches U3.10 (IOL_5B)
- net IO10: now also J3.13 (Pin_13)
- net IO100: now reaches U3.100 (IOT_95)
- net IO100: now also J2.2 (Pin_2)
- net +1V2: now reaches C4.1, U3.11 (VCC)
- net +1V2: now also C16.1, C17.1, C3.1, C6.1, L1.1, R8.2, U3.35 (VCC), U3.61 (VCC), U3.77 (VCC), J6.3 (Pin_3)
- net IO12: now reaches U3.12 (IOL_6A)
- net IO12: now also J3.12 (Pin_12)
- net IO13: now reaches U3.13 (IOL_6B_GBIN7)
- net IO13: now also J3.11 (Pin_11)
- net +3V3: now reaches C7.1, U3.14 (VCCIO_3)
- net +3V3: now also C1.1, C10.1, C11.1, C12.1, C13.1, C14.1, C15.1, C2.1, C5.1, C8.1, C9.1, D1.2 (A), R1.1, R2.1, R3.1, R4.1, R5.1, R6.1, U1.1 (RUN), U1.4 (VIN), U2.3 (~WP~/IO2), U2.7 (~HOLD~/IO3), U2.8 (VCC), U3.22 (VCCIO_3), U3.31 (VCCIO_2), U3.38 (VCCIO_2), U3.50 (VCC_SPI), U3.58 (VCCIO_1), U3.6 (VCCIO_3), U3.67 (VCCIO_1), U3.88 (VCCIO_0), U3.92 (VCCIO_0), J1.1 (Pin_1), J6.2 (Pin_2)
- net IO15: now reaches U3.15 (IOL_7A_GBIN6)
- net IO15: now also J3.10 (Pin_10)
- net IO16: now reaches U3.16 (IOL_7B)
- net IO16: now also J3.9 (Pin_9)
- net GND: now reaches U3.17 (GND)
- net GND: now also C1.2, C10.2, C11.2, C12.2, C13.2, C14.2, C15.2, C16.2, C17.2, C2.2, C3.2, C4.2, C5.2, C6.2, C7.2, C8.2, C9.2, R7.2, U1.2 (GND), U2.4 (GND), U3.23 (GND), U3.32 (GND), U3.39 (GND), U3.47 (GND), U3.5 (GND), U3.55 (GND), U3.70 (GND), U3.84 (GND), U3.98 (GND), J1.2 (Pin_2), J6.1 (Pin_1)
- net IO18: now reaches U3.18 (IOL_8A)
- net IO18: now also J3.8 (Pin_8)
- net IO19: now reaches U3.19 (IOL_8B)
- net IO19: now also J3.7 (Pin_7)
- net IO2: now reaches U3.2 (IOL_1B)
- net IO2: now also J3.19 (Pin_19)
- net IO20: now reaches U3.20 (IOL_10A)
- net IO20: now also J3.6 (Pin_6)
- net IO21: now reaches U3.21 (IOL_10B)
- net IO21: now also J3.5 (Pin_5)
- net IO24: now reaches U3.24 (IOL_12A)
- net IO24: now also J3.4 (Pin_4)
- net IO25: now reaches U3.25 (IOL_12B)
- net IO25: now also J3.3 (Pin_3)
- net IO26: now reaches U3.26 (IOB_26)
- net IO26: now also J4.12 (Pin_12)
- net IO27: now reaches U3.27 (IOB_27)
- net IO27: now also J4.11 (Pin_11)
- net IO28: now reaches U3.28 (IOB_28)
- net IO28: now also J4.10 (Pin_10)
- net IO29: now reaches U3.29 (IOB_29)
- net IO29: now also J4.9 (Pin_9)
- net IO3: now reaches U3.3 (IOL_2A)
- net IO3: now also J3.18 (Pin_18)
- net IO30: now reaches U3.30 (IOB_30)
- net IO30: now also J4.8 (Pin_8)
- net IO33: now reaches U3.33 (IOB_35_GBIN5)
- net IO33: now also J4.7 (Pin_7)
- net IO34: now reaches U3.34 (IOB_36_GBIN4)
- net IO34: now also J4.6 (Pin_6)
- net IO36: now reaches U3.36 (IOB_34)
- net IO36: now also J4.5 (Pin_5)
- net IO37: now reaches U3.37 (IOB_37)
- net IO37: now also J4.4 (Pin_4)
- net IO4: now reaches U3.4 (IOL_2B)
- net IO4: now also J3.17 (Pin_17)
- net IO40: now reaches U3.40 (IOB_41)
- net IO40: now also J4.3 (Pin_3)
- net IO41: now reaches U3.41 (IOB_42_CBSEL0)
- net IO41: now also J4.2 (Pin_2)
- net IO43: now reaches U3.42 (IOB_43_CBSEL1)
- net IO43: now also J4.1 (Pin_1)
- net CDONE: now reaches U3.43 (CDONE)
- net CDONE: now also R1.2, J1.5 (Pin_5)
- net CRESET: now reaches U3.44 (CRESET_B)
- net CRESET: now also R2.2, J1.7 (Pin_7)
- net SPI_OUT: now reaches U3.45 (IOB_44_SDO)
- net SPI_OUT: now also R4.2, U2.5 (SI/IO0), J1.10 (Pin_10)
- net SPI_IN: now reaches U3.46 (IOB_45_SDI)
- net SPI_IN: now also R3.2, U2.2 (SO/IO1), J1.9 (Pin_9)
- net SPI_SCK: now reaches U3.48 (IOB_46_SCK)
- net SPI_SCK: now also R5.2, U2.6 (SCK), J1.8 (Pin_8)
- net SPI_CS: now reaches U3.49 (IOB_47_SS)
- net SPI_CS: now also R6.2, U2.1 (~CS), J1.6 (Pin_6)
- net IO51: now reaches U3.51 (IOR_52)
- net IO51: now also J5.19 (Pin_19)
- net IO52: now reaches U3.52 (IOR_53)
- net IO52: now also J5.18 (Pin_18)
- net IO53: now reaches U3.53 (IOR_54)
- net IO53: now also J5.17 (Pin_17)
- net IO54: now reaches U3.54 (IOR_55)
- net IO54: now also J5.16 (Pin_16)
- net IO56: now reaches U3.56 (IOR_56)
- net IO56: now also J5.15 (Pin_15)
- net IO57: now reaches U3.57 (IOR_57)
- net IO57: now also J5.14 (Pin_14)
- net IO59: now reaches U3.59 (IOR_58)
- net IO59: now also J5.13 (Pin_13)
- net IO60: now reaches U3.60 (IOR_59)
- net IO60: now also J5.12 (Pin_12)
- net IO62: now reaches U3.62 (IOR_60_GBIN3)
- net IO62: now also J5.11 (Pin_11)
- net IO63: now reaches U3.63 (IOR_61_GBIN2)
- net IO63: now also J5.10 (Pin_10)
- net IO64: now reaches U3.64 (IOR_63)
- net IO64: now also J5.9 (Pin_9)
- net IO65: now reaches U3.65 (IOR_64)
- net IO65: now also J5.8 (Pin_8)
- net IO66: now reaches U3.66 (IOR_65)
- net IO66: now also J5.7 (Pin_7)
- net IO68: now reaches U3.68 (IOR_67)
- net IO68: now also J5.6 (Pin_6)
- net IO69: now reaches U3.69 (IOR_68)
- net IO69: now also J5.5 (Pin_5)
- net IO7: now reaches U3.7 (IOL_3A)
- net IO7: now also J3.16 (Pin_16)
- net IO71: now reaches U3.71 (IOR_69)
- net IO71: now also J5.4 (Pin_4)
- net IO72: now reaches U3.72 (IOR_70)
- net IO72: now also J5.3 (Pin_3)
- net IO73: now reaches U3.73 (IOR_71)
- net IO73: now also J5.2 (Pin_2)
- net IO74: now reaches U3.74 (IOR_72)
- net IO74: now also J5.1 (Pin_1)
- net IO78: now reaches U3.78 (IOT_73)
- net IO78: now also J2.20 (Pin_20)
- net IO79: now reaches U3.79 (IOT_74)
- net IO79: now also J2.19 (Pin_19)
- net IO8: now reaches U3.8 (IOL_3B)
- net IO8: now also J3.15 (Pin_15)
- net IO80: now reaches U3.80 (IOT_75)
- net IO80: now also J2.18 (Pin_18)
- net IO81: now reaches U3.81 (IOT_77)
- net IO81: now also J2.17 (Pin_17)
- net IO82: now reaches U3.82 (IOT_78)
- net IO82: now also J2.16 (Pin_16)
- net IO83: now reaches U3.83 (IOT_79)
- net IO83: now also J2.15 (Pin_15)
- net IO85: now reaches U3.85 (IOT_80)
- net IO85: now also J2.14 (Pin_14)
- net IO86: now reaches U3.86 (IOT_81)
- net IO86: now also J2.13 (Pin_13)
- net IO87: now reaches U3.87 (IOT_82)
- net IO87: now also J2.12 (Pin_12)
- net IO89: now reaches U3.89 (IOT_84_GBIN1)
- net IO89: now also J2.11 (Pin_11)
- net IO9: now reaches U3.9 (IOL_5A)
- net IO9: now also J3.14 (Pin_14)
- net IO90: now reaches U3.90 (IOT_85_GBIN0)
- net IO90: now also J2.10 (Pin_10)
- net IO91: now reaches U3.91 (IOT_86)
- net IO91: now also J2.9 (Pin_9)
- net IO93: now reaches U3.93 (IOT_87)
- net IO93: now also J2.8 (Pin_8)
- net IO94: now reaches U3.94 (IOT_88)
- net IO94: now also J2.7 (Pin_7)
- net IO95: now reaches U3.95 (IOT_89)
- net IO95: now also J2.6 (Pin_6)
- net IO96: now reaches U3.96 (IOT_90)
- net IO96: now also J2.5 (Pin_5)
- net IO97: now reaches U3.97 (IOT_91)
- net IO97: now also J2.4 (Pin_4)
- net IO99: now reaches U3.99 (IOT_93)
- net IO99: now also J2.3 (Pin_3)
- no-connect marks 0 -> 15
Other:
- moved on the sheet: R1, R2, R3, R4, R5, R6
