File: hardware/ice40HX1Kboard/ice40HX1Kboard/ice40HX1Kboard/ice40HX1Kboard.kicad_pcb (KiCad board)
At the start: 2 copper layers, 124.5 x 96.5 mm, 36 parts, among them J1 Conn_02x05_Odd_Even, J2 Conn_01x20_Male, J3 Conn_01x20_Male, J4 Conn_01x20_Male, J5 Conn_01x20_Male, J6 Conn_01x03_Male, U1 LTC3406ES5, U2 AT25SF081-SSHD-X, U3 ICE40HX1K-VQ100(VQFP100)

Commit message: HX1Kboard improvement
Routing:
- net GND: track 62.6 -> 33.4 mm, vias 272 -> 275
- net IO54: track 35.9 -> 33.1 mm
- net IO64: track 30.7 -> 28.5 mm
- net IO7: track 35.6 -> 33.5 mm

Commit message: updated PCB settings
Other:
- rule pad_to_mask_clearance: 0.05 -> 0
Changed lines of the file:
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@@
     (pad_size 1.524 1.524)
     (pad_drill 0.762)
-    (pad_to_mask_clearance 0.05)
+    (pad_to_mask_clearance 0)
     (aux_axis_origin 0 0)
     (visible_elements 7FFFFFFF)
