File: hardware/LP1Kboard/LP1Kboard/LP1Kboard/LP1Kboard.sch (KiCad schematic (older format))
At the start: 30 parts, among them J1 Conn_02x05_Odd_Even, J6 Conn_01x03_Male, U1 LTC3406ES5, U2 AT25SF081-SSHD-X, U3 ICE40LP1K-CM36

Commit message: LP1K + HX1Kcap boards
Parts:
- U3: footprint Package_CSP:WLCSP-36_2.82x2.67mm_Layout6x6_P0.4mm -> kifootp:ice40-CM36-WLCSP-36_2.82x2.67mm_Layout6x6_P0.4mm
Changed lines of the file:
@@
 EESchema Schematic File Version 4
+LIBS:LP1Kboard-cache
 EELAYER 30 0
 EELAYER END
@@
 F 0 "U3" H 5975 3265 50  0000 C CNN
 F 1 "ICE40LP1K-CM36" H 5975 3174 50  0000 C CNN
-F 2 "Package_CSP:WLCSP-36_2.82x2.67mm_Layout6x6_P0.4mm" H 6150 3400 50  0001 C CNN
+F 2 "kifootp:ice40-CM36-WLCSP-36_2.82x2.67mm_Layout6x6_P0.4mm" H 6150 3400 50  0001 C CNN
 F 3 "" H 6000 2450 50  0001 C CNN
 	1    6000 2450
