File: hardware/LEDregul/LEDregul/LEDregul/LEDregul.sch (KiCad schematic (older format))
At the start: 1 part, among them J4 Conn_01x20_Female

Commit message: started new boards
Parts:
- added BT1: Battery_Cell, symbol Device:Battery_Cell
- added C1: 1uF, symbol Device:C
- added C2: 10uF, symbol Device:C
- added D1, D2, D3, D4, D5: LED, symbol Device:LED
- added J1: Conn_02x04_Odd_Even, symbol Connector_Generic:Conn_02x04_Odd_Even
- added L1: L, symbol Device:L
- added R1: R, symbol Device:R
- added U1: FAN5341, symbol Regulator_Switching:LTC3429
- added X1: SiT1569, symbol Oscillator:XO32
Connections:
- net at J4.11 (Pin_11): now also X1.3 (OUT)
- net at J4.17 (Pin_17): now also U1.4 (~SHDN)
- new net: L1.2, U1.1 (SW)
- new net: D5.1 (K), R1.1, U1.3 (FB)
- new net: C1.1, D1.2 (A), U1.5 (VOUT)
- new net: D1.1 (K), D2.2 (A)
- new net: D2.1 (K), D3.2 (A)
- new net: D3.1 (K), D4.2 (A)
- new net: D4.1 (K), D5.2 (A)
- new net +3V3: BT1.1 (+), C2.1, J1.2 (Pin_2), J1.4 (Pin_4), J1.6 (Pin_6), J1.8 (Pin_8), L1.1, U1.6 (VIN), X1.4 (V+)
- new net GND: BT1.2 (-), C1.2, C2.2, J1.1 (Pin_1), J1.3 (Pin_3), J1.5 (Pin_5), J1.7 (Pin_7), R1.2, U1.2 (GND), X1.2 (GND)

Commit message: LEDregul I board
Parts:
- added C3, C4, C7: 1uF, Capacitor_SMD:C_1206_3216Metric, symbol Device:C
- added C5, C6, C8: 10uF, Capacitor_SMD:C_1206_3216Metric, symbol Device:C
- added D10, D11, D12, D13, D14, D15, D16, D17, D18, D19, D20, D6, D7, D8, D9: LED, LED_SMD:LED_1206_3216Metric, symbol Device:LED
- added J2: Conn_01x04_Male, Connector_PinHeader_2.54mm:PinHeader_1x04_P2.54mm_Vertical, symbol Connector:Conn_01x04_Male
- added L2, L3, L4: L, Inductor_SMD:L_1812_4532Metric, symbol Device:L
- added R2, R3, R4: R, Resistor_SMD:R_0402_1005Metric, symbol Device:R
- added U2, U3, U4: FAN5341, kifootp:FAN5341, symbol kilib:FAN5341
- BT1: footprint (none) -> kifootp:CR2032
- C1, C2: footprint (none) -> Capacitor_SMD:C_1206_3216Metric
- D1, D2, D3, D4, D5: footprint (none) -> LED_SMD:LED_1206_3216Metric
- J1: footprint (none) -> Connector_PinHeader_2.54mm:PinHeader_2x04_P2.54mm_Vertical
- L1: footprint (none) -> Inductor_SMD:L_1812_4532Metric
- R1: footprint (none) -> Resistor_SMD:R_0402_1005Metric
- U1: footprint (none) -> kifootp:FAN5341; symbol Regulator_Switching:LTC3429 -> kilib:FAN5341
- X1: value SiT1569 -> SiT1534; footprint (none) -> kifootp:SiT1534
Connections:
- net +3V3: now also U1.2 (VIN), C5.1, C6.1, C8.1, J2.3 (Pin_3), J2.4 (Pin_4), L2.1, L3.1, L4.1, U2.2 (VIN), U3.2 (VIN), U4.2 (VIN); no longer BT1.1 (+), U1.6 (VIN)
- net GND: now also U1.6 (GND), C3.2, C4.2, C5.2, C6.2, C7.2, C8.2, R2.2, R3.2, R4.2, U2.6 (GND), U3.6 (GND), U4.6 (GND); no longer U1.2 (GND)
- net at U1.1 (VOUT): now also C1.1, D1.2 (A); no longer L1.2
- net at D5.1 (K), R1.1: now also U1.4 (FB); no longer U1.3 (FB)
- net at J4.17 (Pin_17): now also U1.3 (EN); no longer U1.4 (~SHDN)
- net C3: now reaches J4.10 (Pin_10)
- net C3: now also U2.3 (EN)
- net C1: now reaches J4.8 (Pin_8)
- net C1: now also U4.3 (EN)
- net C2: now reaches J4.9 (Pin_9)
- net C2: now also U3.3 (EN)
- new net: BT1.1 (+), J2.1 (Pin_1), J2.2 (Pin_2)
- new net: L1.2, U1.5 (SW)
- new net: C4.1, D11.2 (A), U3.1 (VOUT)
- new net: D15.1 (K), R3.1, U3.4 (FB)
- new net: L3.2, U3.5 (SW)
- new net: D11.1 (K), D12.2 (A)
- new net: D12.1 (K), D13.2 (A)
- new net: D13.1 (K), D14.2 (A)
- new net: D14.1 (K), D15.2 (A)
- new net: C3.1, D6.2 (A), U2.1 (VOUT)
- new net: D10.1 (K), R2.1, U2.4 (FB)
- new net: L2.2, U2.5 (SW)
- new net: D6.1 (K), D7.2 (A)
- new net: D7.1 (K), D8.2 (A)
- new net: D8.1 (K), D9.2 (A)
- new net: D10.2 (A), D9.1 (K)
- new net: C7.1, D16.2 (A), U4.1 (VOUT)
- new net: D20.1 (K), R4.1, U4.4 (FB)
- new net: L4.2, U4.5 (SW)
- new net: D16.1 (K), D17.2 (A)
- new net: D17.1 (K), D18.2 (A)
- new net: D18.1 (K), D19.2 (A)
- new net: D19.1 (K), D20.2 (A)
- no-connect marks 19 -> 16
