File: hardware/nrf52810/nrf52810/nrf52810/nrf52810.kicad_pcb (KiCad board)
At the start: 2 copper layers, 65.2 x 35.1 mm, 17 parts, among them J1 Conn_01x04_Female, J2 Conn_01x16_Male, J3 Conn_01x04_Male, U1 nRF52810-QCxx, Y1 Crystal_GND24

Commit message: nRF52 board + capSense
Parts:
- Y1: footprint Crystal:Crystal_SMD_3225-4Pin_3.2x2.5mm_HandSoldering -> Crystal:Crystal_SMD_3225-4Pin_3.2x2.5mm
- moved C2 2.42 mm to (123.4, 71.4), turned to 270 degrees
- moved C1 1.95 mm to (127.3, 67.3)
- moved Y1 0.69 mm to (126.2, 69.8)
Routing:
- net GND: track 28.9 -> 24.4 mm, vias 75 -> 79
- net Net-(C2-Pad1): track 12.4 -> 9.35 mm
- net Net-(C1-Pad1): track 12.2 -> 9.87 mm
