File: hardware/RFboard1/RFboard1/RFboard1/RFboard1.kicad_pcb (KiCad board)
At the start: 2 copper layers, 37 x 53 mm, 19 parts, among them J1 Conn_01x04_Male, J3 Conn_02x04_Odd_Even, J4 Conn_01x20_Female, Q1 2N7002, Q2 2N7002, Q3 2N7002, Q4 2N7002, Q5 2N7002

Commit message: RFboard
Parts:
- removed BT1: Battery_Cell, kifootp:CR2032
- removed D1, D2, D3, D4, D5: LED, LED_SMD:LED_1206_3216Metric
- removed Q1, Q4, Q5: 2N7002, Package_TO_SOT_SMD:SOT-23
- removed R1, R2, R3, R4: 10 kOhm, Resistor_SMD:R_0402_1005Metric
- added C1: C, Capacitor_SMD:C_1206_3216Metric, F.Cu at (87.1, 56.1)
- added L3: L, Inductor_SMD:L_1210_3225Metric, F.Cu at (93.7, 53.6)
- added R7: R, Resistor_SMD:R_1206_3216Metric, F.Cu at (81.0, 53.8)
- added R8: R, Resistor_SMD:R_1206_3216Metric, F.Cu at (91.9, 47.2)
- J1: value Conn_01x04_Male -> Conn_01x05_Male; footprint Connector_PinSocket_2.54mm:PinSocket_1x04_P2.54mm_Vertical -> Connector_PinHeader_2.54mm:PinHeader_1x05_P2.54mm_Vertical
- R5: value 10 kOhm -> R; footprint Resistor_SMD:R_0402_1005Metric -> Resistor_SMD:R_1206_3216Metric
- moved J3 30.4 mm to (91.4, 37.3), turned to 180 degrees
- moved R5 29.5 mm to (81.3, 61.2), turned to 180 degrees
- moved J1 17.8 mm to (87.8, 61.0), turned to 90 degrees
- moved Q3 5.85 mm to (80.5, 39.4), turned to 90 degrees
- moved Q2 2.37 mm to (80.0, 45.7), turned to 90 degrees
Connections:
- J1 pad 1: +3V3 -> Net-(C1-Pad1)
- J1 pad 2: +3V3 -> Net-(J1-Pad2)
- J1 pad 3: Net-(BT1-Pad1) -> Net-(J1-Pad3)
- J1 pad 4: Net-(BT1-Pad1) -> Net-(J1-Pad4)
- Q2 pad 1: Net-(J4-Pad14) -> Net-(J4-Pad13)
- Q3 pad 1: Net-(J4-Pad15) -> Net-(J4-Pad14)
- R5 pad 1: Net-(D5-Pad1) -> Net-(C1-Pad1)
Routing:
- net +3V3: track 73.2 -> 17.9 mm
- net Net-(BT1-Pad1): track 54.5 -> 0.00 mm
- net Net-(D1-Pad2): track 25.0 -> 0.00 mm, vias 2 -> 0
- net Net-(D5-Pad2): track 22.7 -> 0.00 mm, vias 2 -> 0
- net Net-(D4-Pad2): track 17.8 -> 0.00 mm, vias 2 -> 0
- net Net-(C1-Pad1): track 0.00 -> 14.9 mm
- net Net-(J1-Pad2): track 0.00 -> 13.0 mm
- net Net-(J4-Pad15): track 12.2 -> 0.00 mm
- net Net-(J4-Pad16): track 11.6 -> 1.34 mm
- net Net-(Q2-Pad2): track 15.7 -> 5.63 mm, vias 2 -> 0
- net Net-(J4-Pad17): track 7.78 -> 0.00 mm
- net Net-(Q3-Pad2): track 18.9 -> 12.8 mm, vias 2 -> 0
- net Net-(D4-Pad1): track 2.77 -> 0.00 mm
- net Net-(D3-Pad1): track 2.77 -> 0.00 mm
- net Net-(D1-Pad1): track 2.72 -> 0.00 mm
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