File: hardware/mcu/stdAtmelUSB/stdAtmelUSB/stdAtmelUSB/stdAtmelUSB.kicad_pcb (KiCad board)
At the start: 2 copper layers, 37 x 53 mm, 22 parts, among them J1 Conn_01x20_Female, J5 Conn_01x06_Male, U3 LTC3406ES5, U4 MAX40200AUK, U8 ATSAMD11D14A-SS, X1 USBFCI_10103594_MILL

Commit message: std boards skeletons
Parts:
- moved C9 122.3 mm to (92.7, 71.2)
- moved U3 122.3 mm to (97.4, 73.2)
- moved U4 122.3 mm to (97.7, 68.7)
- moved C3 122.3 mm to (93.8, 67.0)
- moved C6 122.3 mm to (88.3, 74.2)
- moved C7 122.3 mm to (89.3, 71.5)
- moved C8 122.3 mm to (93.8, 69.0)
- moved L2 122.3 mm to (92.5, 74.0)
- moved R3 122.3 mm to (84.9, 74.5)
- moved R4 122.3 mm to (90.9, 69.0)
- moved X1 56.6 mm to (107.9, 43.8), turned to 90 degrees
- moved D6 56.0 mm to (86.4, 60.3), turned to 90 degrees
- moved R15 54.9 mm to (85.3, 57.1), turned to 0 degrees
- moved C1 52.9 mm to (86.4, 54.3), turned to 270 degrees
- moved R1 52.5 mm to (92.7, 53.8)
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Routing:
- added copper zone on B.Cu, net GND
- added copper zone on F.Cu, net GND

Commit message: std Atmel USB skeletons
Routing:
- net +3V3: track 0.00 -> 56.5 mm, vias 0 -> 1
- net nrf_tx: track 0.00 -> 31.9 mm
- net nrf_rx: track 0.00 -> 31.4 mm
- net uart_rx: track 0.00 -> 31.0 mm, vias 0 -> 2
- net fpga_cdone: track 0.00 -> 30.8 mm
- net fpga_reset: track 0.00 -> 30.1 mm
- net spi_clk: track 0.00 -> 27.1 mm
- net uart_tx: track 0.00 -> 26.7 mm, vias 0 -> 2
- net uart_fpga_rx_2: track 0.00 -> 24.1 mm
- net uart_fpga_tx_2: track 0.00 -> 23.5 mm
- net spi_mosi: track 0.00 -> 21.8 mm
- net spi_miso: track 0.00 -> 21.2 mm
- net spi_ss: track 0.00 -> 19.1 mm
- net led_mcu: track 0.00 -> 16.7 mm
- net swd_rst: track 0.00 -> 16.6 mm
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
Commit message: std Atmel USB skeletons
Parts:
- moved C9 15.3 mm to (98.2, 57.0), turned to 0 degrees
- moved C6 14.4 mm to (102.6, 75.7)
- moved R3 14.3 mm to (98.3, 69.5), turned to 90 degrees
- moved L2 11.0 mm to (103.5, 73.2), turned to 90 degrees
- moved C7 11.0 mm to (93.5, 61.3), turned to 90 degrees
- moved C8 9.84 mm to (97.9, 60.0), turned to 0 degrees
- moved C3 8.39 mm to (102.2, 68.0), turned to 0 degrees
- moved R4 8.07 mm to (98.4, 72.0), turned to 270 degrees
- moved U4 5.97 mm to (96.3, 62.9), turned to 0 degrees
- moved U3 4.09 mm to (100.7, 70.8), turned to 90 degrees
Routing:
- net +5V: track 0.00 -> 48.4 mm, vias 0 -> 2
- net Net-(C6-Pad1): track 0.00 -> 28.9 mm
- net +3V3: track 56.5 -> 69.3 mm
- net Net-(R3-Pad1): track 0.00 -> 3.04 mm
- net Net-(L2-Pad2): track 0.00 -> 1.80 mm

Commit message: std Atmel USB skeletons
Routing:
- net Net-(C6-Pad1): track 28.9 -> 35.9 mm
- net +5V: track 48.4 -> 46.8 mm
- net GND: vias 0 -> 330
