File: hardware/mcu/nrf52/nrf52/nrf52.sch (KiCad schematic (older format))
At the start: 11 parts

Commit message: std nRF52 skeleton
Parts:
- added J?: Conn_01x20_Male, symbol Connector:Conn_01x20_Male
- added J?: Conn_01x20_Female, symbol Connector:Conn_01x20_Female
- added J?: Conn_01x04_Male, symbol Connector:Conn_01x04_Male
Connections:
- net +3V3: now also J?.19 (Pin_19), J?.19 (Pin_19)
- net GND: now also J?.1 (Pin_1), J?.1 (Pin_1), J?.15 (Pin_15), J?.15 (Pin_15), J?.18 (Pin_18), J?.18 (Pin_18), J?.20 (Pin_20), J?.20 (Pin_20), J?.4 (Pin_4), J?.4 (Pin_4), J?.8 (Pin_8), J?.8 (Pin_8)
Changed lines of the file:
@@
 Wire Wire Line
 	6700 6050 7100 6050
+$Comp
+L Connector:Conn_01x20_Male J?
+U 1 1 5EA6E6FC
+P 1700 4600
+F 0 "J?" H 1808 5681 50  0000 C CNN
+F 1 "Conn_01x20_Male" H 1808 5590 50  0000 C CNN
+F 2 "" H 1700 4600 50  0001 C CNN
+F 3 "~" H 1700 4600 50  0001 C CNN
+	1    1700 4600
+	1    0    0    -1
+$EndComp
+$Comp
+L Connector:Conn_01x20_Female J?
+U 1 1 5EA6FAD6
+P 1550 4600
+F 0 "J?" H 1578 4576 50  0000 L CNN
+F 1 "Conn_01x20_Female" H 1578 4485 50  0000 L CNN
+F 2 "" H 1550 4600 50  0001 C CNN
+F 3 "~" H 1550 4600 50  0001 C CNN
+	1    1550 4600
+	1    0    0    -1
+$EndComp
+$Comp
+L power:+3V3 #PWR?
+U 1 1 5EA812AE
+P 2350 3300
+F 0 "#PWR?" H 2350 3150 50  0001 C CNN
+F 1 "+3V3" H 2365 3473 50  0000 C CNN
+F 2 "" H 2350 3300 50  0001 C CNN
+F 3 "" H 2350 3300 50  0001 C CNN
+	1    2350 3300
+	1    0    0    -1
+$EndComp
+Wire Wire Line
+	1900 5500 2350 5500
+Wire Wire Line
+	2350 3300 2350 5500
+$Comp
+L power:GND #PWR?
+U 1 1 5EA84AA8
+P 2200 5950
+F 0 "#PWR?" H 2200 5700 50  0001 C CNN
+F 1 "GND" H 2205 5777 50  0000 C CNN
+F 2 "" H 2200 5950 50  0001 C CNN
+F 3 "" H 2200 5950 50  0001 C CNN
+	1    2200 5950
+	1    0    0    -1
+$EndComp
+Wire Wire Line
+	2200 5950 2200 5600
+Wire Wire Line
+	1900 5600 2200 5600
+Wire Wire Line
+	2200 5600 2200 5400
+Wire Wire Line
+	2200 3700 1900 3700
+Connection ~ 2200 5600
+Wire Wire Line
+	1900 5400 2200 5400
+Connection ~ 2200 5400
+Wire Wire Line
+	2200 5400 2200 5100
+Wire Wire Line
+	1900 4400 2200 4400
+Connection ~ 2200 4400
+Wire Wire Line
+	2200 4400 2200 4000
+Wire Wire Line
+	1900 4000 2200 4000
+Connection ~ 2200 4000
+Wire Wire Line
+	2200 4000 2200 3700
+Wire Wire Line
+	1900 5100 2200 5100
+Connection ~ 2200 5100
+Wire Wire Line
+	2200 5100 2200 4400
+$Comp
+L power:GND #PWR?
+U 1 1 5EA8BB06
+P 1100 5950
+F 0 "#PWR?" H 1100 5700 50  0001 C CNN
+F 1 "GND" H 1105 5777 50  0000 C CNN
+F 2 "" H 1100 5950 50  0001 C CNN
+F 3 "" H 1100 5950 50  0001 C CNN
+	1    1100 5950
+	1    0    0    -1
+$EndComp
+$Comp
+L power:+3V3 #PWR?
+U 1 1 5EA8FE7D
+P 1000 3250
+F 0 "#PWR?" H 1000 3100 50  0001 C CNN
+F 1 "+3V3" H 1015 3423 50  0000 C CNN
+F 2 "" H 1000 3250 50  0001 C CNN
+F 3 "" H 1000 3250 50  0001 C CNN
+	1    1000 3250
+	1    0    0    -1
+$EndComp
+Wire Wire Line
+	1350 5500 1000 5500
+Wire Wire Line
+	1000 3250 1000 5500
+Wire Wire Line
+	1100 3700 1350 3700
+Wire Wire Line
+	1100 3700 1100 4000
+Wire Wire Line
+	1350 5600 1100 5600
+Connection ~ 1100 5600
+Wire Wire Line
+	1100 5600 1100 5950
+Wire Wire Line
+	1100 5400 1350 5400
+Connection ~ 1100 5400
+Wire Wire Line
+	1100 5400 1100 5600
+Wire Wire Line
+	1350 5100 1100 5100
+Connection ~ 1100 5100
+Wire Wire Line
+	1100 5100 1100 5400
+Wire Wire Line
+	1100 4400 1350 4400
+Connection ~ 1100 4400
+Wire Wire Line
+	1100 4400 1100 5100
+Wire Wire Line
+	1350 4000 1100 4000
+Connection ~ 1100 4000
+Wire Wire Line
+	1100 4000 1100 4400
+$Comp
+L Connector:Conn_01x04_Male J?
+U 1 1 5EA9CF97
+P 9700 1700
+F 0 "J?" H 9672 1582 50  0000 R CNN
+F 1 "Conn_01x04_Male" H 9672 1673 50  0000 R CNN
+F 2 "" H 9700 1700 50  0001 C CNN
+F 3 "~" H 9700 1700 50  0001 C CNN
+	1    9700 1700
+	-1   0    0    1
+$EndComp
 $EndSCHEMATC

Commit message: std nRF52 skeleton
Parts:
- J1: renamed from J?; footprint (none) -> Connector_PinHeader_2.54mm:PinHeader_1x20_P2.54mm_Horizontal
- J2: renamed from J?; footprint (none) -> Connector_PinSocket_2.54mm:PinSocket_1x20_P2.54mm_Horizontal
- J3: renamed from J?; footprint (none) -> Connector_PinHeader_2.54mm:PinHeader_1x04_P2.54mm_Vertical
- gave numbers to parts that had none: 11
Connections:
- net +3V3: now also J3.4 (Pin_4)
- net GND: now also J3.1 (Pin_1)
- net at U1.15 (SIO_09/NFC1): now also J1.2 (Pin_2)
- net at U1.17 (SIO_08): now also J1.3 (Pin_3)
- net at U1.28 (SIO_13): now also J2.17 (Pin_17)
- net at U1.29 (SIO_15): now also J2.16 (Pin_16)
- net at U1.30 (SIO_17): now also J2.14 (Pin_14)
- net at U1.31 (SIO_19): now also D3.2 (A)
- net at U1.32 (SIO_31/AIN7): now also J2.13 (Pin_13)
- net at U1.33 (SIO_30/AIN6): now also J2.12 (Pin_12)
- net at U1.34 (SIO_29/AIN5): now also J2.11 (Pin_11)
- net at U1.35 (SIO_28/AIN4): now also J2.10 (Pin_10)
- net at U1.36 (SIO_27): now also J2.9 (Pin_9)
- net at U1.5 (SWDIO): now also J3.2 (Pin_2)
- net at U1.6 (SWDCLK): now also J3.3 (Pin_3)
- net at U1.7 (SIO_21): now also D1.2 (A)
- net at U1.8 (SIO_20): now also D2.2 (A)
- net at U1.9 (SIO_18): now also D4.2 (A)
- no-connect marks 0 -> 34
