File: hardware/mcu/nrf52/nrf52/nrf52.kicad_pcb (KiCad board)
At the start: 2 copper layers, 46.9 x 59.8 mm, 14 parts, among them J1 Conn_01x20_Female, J2 Conn_01x20_Male, J3 Conn_01x04_Male, U1 BL652

Commit message: std nRF52 skeleton
Other:
- rule pad_to_mask_clearance: 0.051 -> 0
Changed lines of the file:
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@@
     (pad_size 1.524 1.524)
     (pad_drill 0.762)
-    (pad_to_mask_clearance 0.051)
-    (solder_mask_min_width 0.25)
+    (pad_to_mask_clearance 0)
     (aux_axis_origin 0 0)
     (visible_elements FFFFFF7F)
