File: hardware/mcu/esp8266/esp8266/esp8266.sch (KiCad schematic (older format))
At the start: 13 parts, among them J1 Conn_01x20_Female, J2 Conn_01x20_Male, J3 Conn_01x04_Male

Commit message: some esp8266 skeleton
Parts:
- removed D4: LED, Capacitor_SMD:C_1206_3216Metric, symbol Device:LED
- removed R4: 10kOhm, Resistor_SMD:R_0402_1005Metric, symbol Device:R
- added C3: 0.1uF, Capacitor_SMD:C_0402_1005Metric, symbol Device:C
- added R10, R11, R12, R5, R8, R9: 10kOhm, Resistor_SMD:R_0402_1005Metric, symbol Device:R
- added R6, R7: 1kOhm, Resistor_SMD:R_0402_1005Metric, symbol Device:R
- added U1: ESP-WROOM-02, RF_Module:ESP-WROOM-02, symbol RF_Module:ESP-WROOM-02
Connections:
- net labels added: esp8266_en, esp_8266_nrst, led1, led2, led3, miso, mosi, pull_down_io15, pull_up_io14, pull_up_io2, uart_rx, uart_sel, uart_tx
- wire segments 76 -> 86
- no-connect marks 16 -> 21
