File: hardware/power/power3X/power3X/power3X.kicad_pcb (KiCad board)
At the start: 2 copper layers, 37 x 53 mm, 22 parts, among them J1 Conn_01x20_Female, J5 Conn_01x06_Male, U3 LTC3406ES5, U4 MAX40200AUK, U8 ATSAMD11D14A-SS, X1 USBFCI_10103594_MILL

Commit message: some power skeleton
Parts:
- removed C27: 4.7uF, Capacitor_SMD:C_0402_1005Metric
- removed C28, C8: 0.1uF, Capacitor_SMD:C_0402_1005Metric
- removed C9: 10uF, Capacitor_SMD:C_0603_1608Metric
- removed D6: LED, LED_SMD:LED_1206_3216Metric
- removed J5: Conn_01x06_Male, Connector_PinHeader_2.54mm:PinHeader_1x06_P2.54mm_Vertical
- removed L2: 2.2uH, Inductor_SMD:L_0805_2012Metric
- removed R1, R15: 10kOhm, Resistor_SMD:R_0402_1005Metric
- removed R3: 100kOhm, Resistor_SMD:R_0402_1005Metric
- removed R4: 450kOhm, Resistor_SMD:R_0402_1005Metric
- removed U3: LTC3406ES5, Package_TO_SOT_SMD:TSOT-23-5
- removed U4: MAX40200AUK, Package_TO_SOT_SMD:SOT-23-5
- removed U8: ATSAMD11D14A-SS, Package_SO:SOIC-20W_7.5x12.8mm_P1.27mm
- removed X1: USBFCI_10103594_MILL, kifootp:FCI_10103594_MILL
- added BT1: Battery_Cell, kifootp:CR2032, B.Cu at (92.6, 38.8)
- added BT2: Battery_Cell, kifootp:CR2032, B.Cu at (93.8, 68.9)
- added BT3: Battery_Cell, kifootp:CR2032, F.Cu at (92.5, 38.7)
- added BT4: Battery_Cell, kifootp:CR2032, F.Cu at (93.7, 68.8)
- added C5: 0.1uF, Capacitor_SMD:C_0402_1005Metric, F.Cu at (81.7, 73.4)
- added U1: TPS560200, Package_TO_SOT_SMD:SOT-23-5, F.Cu at (77.9, 56.4)
- added U2: MAX40200AUK, Package_TO_SOT_SMD:SOT-23-5, F.Cu at (77.9, 74.7)
- C1: value 0.1uF -> C; footprint Capacitor_SMD:C_0402_1005Metric -> Capacitor_SMD:C_0603_1608Metric
- C2, C3: value 4.7uF -> C
- C4: value 0.1uF -> C
- C6: value 10uF -> 0.1uF; footprint Capacitor_SMD:C_0603_1608Metric -> Capacitor_SMD:C_0402_1005Metric
- C7: value 0.1uF -> 10uF
- J1: value Conn_01x20_Female -> Conn_01x20_Male; moved to B.Cu
- moved J1 48.4 mm to (73.0, 27.8)
- moved C4 30.4 mm to (76.7, 60.3), turned to 270 degrees
- moved C6 28.7 mm to (76.7, 63.2), turned to 270 degrees
- moved C2 27.5 mm to (81.4, 57.1), turned to 0 degrees
- moved C7 23.5 mm to (76.9, 78.0), turned to 0 degrees
- moved C3 23.2 mm to (79.2, 64.3), turned to 270 degrees
- moved C1 9.87 mm to (79.0, 60.8)
Connections:
- C1 pad 1: swd_rst -> Net-(BT1-Pad1)
- C2 pad 1: +3V3 -> Net-(BT1-Pad1)
- C3 pad 1: +5V -> Net-(C3-Pad1)
- C4 pad 1: +3V3 -> Net-(C3-Pad1)
- J1 pad 10: spi_miso -> Net-(J1-Pad10)
- J1 pad 11: spi_ss -> Net-(J1-Pad11)
- J1 pad 12: spi_clk -> Net-(J1-Pad12)
- J1 pad 13: fpga_reset -> Net-(J1-Pad13)
- J1 pad 14: fpga_cdone -> Net-(J1-Pad14)
- J1 pad 16: uart_tx -> Net-(J1-Pad16)
- J1 pad 17: uart_rx -> Net-(J1-Pad17)
- J1 pad 19: +3V3 -> Net-(C3-Pad1)
- J1 pad 2: nrf_tx -> Net-(J1-Pad2)
- J1 pad 3: nrf_rx -> Net-(J1-Pad3)
- J1 pad 6: uart_fpga_rx_2 -> Net-(J1-Pad6)
- J1 pad 7: uart_fpga_tx_2 -> Net-(J1-Pad7)
- J1 pad 9: spi_mosi -> Net-(J1-Pad9)
Routing:
- net +3V3: track 69.3 -> 0.00 mm, vias 1 -> 0
- net Net-(BT2-Pad2): track 0.00 -> 67.9 mm, vias 0 -> 2
- net Net-(BT1-Pad2): track 0.00 -> 63.3 mm
- net Net-(BT3-Pad2): track 0.00 -> 58.6 mm
- net +5V: track 46.8 -> 0.00 mm, vias 2 -> 0
- net Net-(C6-Pad1): track 35.9 -> 0.00 mm
- net nrf_tx: track 31.9 -> 0.00 mm
- net nrf_rx: track 31.4 -> 0.00 mm
- net uart_rx: track 31.0 -> 0.00 mm, vias 2 -> 0
- net fpga_cdone: track 30.8 -> 0.00 mm
- net fpga_reset: track 30.1 -> 0.00 mm
- net spi_clk: track 27.1 -> 0.00 mm
- net uart_tx: track 26.7 -> 0.00 mm, vias 2 -> 0
- net uart_fpga_rx_2: track 24.1 -> 0.00 mm
- net uart_fpga_tx_2: track 23.5 -> 0.00 mm
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
Commit message: some power skeleton
Parts:
- added L1: L, Inductor_SMD:L_0805_2012Metric, F.Cu at (79.8, 59.8)
- added R1: R, Resistor_SMD:R_0402_1005Metric, F.Cu at (76.2, 60.1)
- added R2: R, Resistor_SMD:R_0402_1005Metric, F.Cu at (76.3, 61.8)
- moved C6 12.1 mm to (77.2, 75.2), turned to 90 degrees
- moved C1 9.06 mm to (77.9, 51.9), turned to 180 degrees
- moved C4 4.76 mm to (80.7, 57.6), turned to 90 degrees
- moved C2 4.58 mm to (78.2, 53.8), turned to 180 degrees
- moved C7 3.70 mm to (75.8, 74.5), turned to 90 degrees
- moved C3 2.82 mm to (80.0, 61.6), turned to 180 degrees
- moved C5 2.39 mm to (79.5, 72.4), turned to 180 degrees
- moved U2 1.87 mm to (79.7, 74.8), turned to 180 degrees
- turned U1 to 90 degrees
Connections:
- J1 pad 19: Net-(C3-Pad1) -> Net-(C6-Pad1)
Routing:
- net Net-(BT1-Pad1): track 0.00 -> 58.6 mm, vias 0 -> 1
- net Net-(C3-Pad1): track 0.00 -> 26.6 mm
- net Net-(R1-Pad2): track 0.00 -> 7.56 mm
- net Net-(C6-Pad1): track 0.00 -> 6.53 mm
- net Net-(L1-Pad2): track 0.00 -> 2.43 mm
