File: hardware/power/power3X/power3X/power3X.sch (KiCad schematic (older format))
At the start: 8 parts

Commit message: some power skeleton
Parts:
- added BT? (x4): Battery_Cell, symbol Device:Battery_Cell
- added U?: MAX40200AUK, Package_TO_SOT_SMD:SOT-23-5, symbol Analog_Switch:MAX40200AUK
Connections:
- net GND: now also BT?.2 (-)
- net at C?.1, C?.1, U?.1 (EN)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: now also BT?.1 (+)
- new net: BT?.1 (+), BT?.2 (-) (x3)
Changed lines of the file:
@@
 Wire Wire Line
 	3500 2650 3650 2650
+$Comp
+L Device:Battery_Cell BT?
+U 1 1 5EB2702E
+P 1700 2950
+F 0 "BT?" H 1818 3046 50  0000 L CNN
+F 1 "Battery_Cell" H 1818 2955 50  0000 L CNN
+F 2 "" V 1700 3010 50  0001 C CNN
+F 3 "~" V 1700 3010 50  0001 C CNN
+	1    1700 2950
+	1    0    0    -1
+$EndComp
+$Comp
+L Device:Battery_Cell BT?
+U 1 1 5EB28955
+P 1700 3250
+F 0 "BT?" H 1818 3346 50  0000 L CNN
+F 1 "Battery_Cell" H 1818 3255 50  0000 L CNN
+F 2 "" V 1700 3310 50  0001 C CNN
+F 3 "~" V 1700 3310 50  0001 C CNN
+	1    1700 3250
+	1    0    0    -1
+$EndComp
+$Comp
+L Device:Battery_Cell BT?
+U 1 1 5EB290CE
+P 1700 3550
+F 0 "BT?" H 1818 3646 50  0000 L CNN
+F 1 "Battery_Cell" H 1818 3555 50  0000 L CNN
+F 2 "" V 1700 3610 50  0001 C CNN
+F 3 "~" V 1700 3610 50  0001 C CNN
+	1    1700 3550
+	1    0    0    -1
+$EndComp
+$Comp
+L Device:Battery_Cell BT?
+U 1 1 5EB298E3
+P 1700 3850
+F 0 "BT?" H 1818 3946 50  0000 L CNN
+F 1 "Battery_Cell" H 1818 3855 50  0000 L CNN
+F 2 "" V 1700 3910 50  0001 C CNN
+F 3 "~" V 1700 3910 50  0001 C CNN
+	1    1700 3850
+	1    0    0    -1
+$EndComp
+Wire Wire Line
+	1700 3950 1700 4450
+Wire Wire Line
+	1700 4450 3200 4450
+Wire Wire Line
+	3200 4450 3200 3300
+Wire Wire Line
+	1700 2750 1700 2150
+Wire Wire Line
+	1700 2150 3200 2150
+Wire Wire Line
+	3200 2150 3200 2650
+$Comp
+L Analog_Switch:MAX40200AUK U?
+U 1 1 5EB307BB
+P 8500 2950
+F 0 "U?" H 8500 3317 50  0000 C CNN
+F 1 "MAX40200AUK" H 8500 3226 50  0000 C CNN
+F 2 "Package_TO_SOT_SMD:SOT-23-5" H 8500 3450 50  0001 C CNN
+F 3 "https://datasheets.maximintegrated.com/en/ds/MAX40200.pdf" H 8500 3450 50  0001 C CNN
+	1    8500 2950
+	1    0    0    -1
+$EndComp
 $EndSCHEMATC

Commit message: some power skeleton
Parts:
- added C5, C6: 0.1uF, Capacitor_SMD:C_0402_1005Metric, symbol Device:C
- added C7: 10uF, Capacitor_SMD:C_0402_1005Metric, symbol Device:C
- added J1: Conn_01x20_Male, Connector_PinHeader_2.54mm:PinHeader_1x20_P2.54mm_Horizontal, symbol Connector:Conn_01x20_Male
- BT1, BT2, BT3, BT4: renamed from BT?; footprint (none) -> kifootp:CR2032
- C1: renamed from C?; footprint (none) -> Capacitor_SMD:C_0603_1608Metric
- C2, C3, C4: renamed from C?; footprint (none) -> Capacitor_SMD:C_0402_1005Metric
- gave numbers to parts that had none: 5
Connections:
- net GND: now also U2.2 (GND), C5.2, C6.2, C7.2, J1.1 (Pin_1), J1.15 (Pin_15), J1.18 (Pin_18), J1.20 (Pin_20), J1.4 (Pin_4), J1.8 (Pin_8)
- net at C3.1, C4.1, L1.1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: now also U2.1 (VDD), U2.3 (EN), C5.1, J1.19 (Pin_19)
- net at U2.5 (OUT): now also C6.1, C7.1
- no-connect marks 0 -> 13

Commit message: some power skeleton
Parts:
- L1: footprint (none) -> Inductor_SMD:L_0805_2012Metric
- R1, R2: footprint (none) -> Resistor_SMD:R_0402_1005Metric
Connections:
- net at C3.1, C4.1, C5.1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: no longer J1.19 (Pin_19)
- net at C6.1, C7.1, U2.5 (OUT): now also J1.19 (Pin_19)
Changed lines of the file:
@@
 F 0 "L1" V 4369 2650 50  0000 C CNN
 F 1 "L" V 4460 2650 50  0000 C CNN
-F 2 "" H 4550 2650 50  0001 C CNN
+F 2 "Inductor_SMD:L_0805_2012Metric" H 4550 2650 50  0001 C CNN
 F 3 "~" H 4550 2650 50  0001 C CNN
 	1    4550 2650
@@
 F 0 "R2" H 6020 2996 50  0000 L CNN
 F 1 "R" H 6020 2905 50  0000 L CNN
-F 2 "" V 5880 2950 50  0001 C CNN
+F 2 "Resistor_SMD:R_0402_1005Metric" V 5880 2950 50  0001 C CNN
 F 3 "~" H 5950 2950 50  0001 C CNN
 	1    5950 2950
@@
 F 0 "R1" H 5520 3696 50  0000 L CNN
 F 1 "R" H 5520 3605 50  0000 L CNN
-F 2 "" V 5380 3650 50  0001 C CNN
+F 2 "Resistor_SMD:R_0402_1005Metric" V 5380 3650 50  0001 C CNN
 F 3 "~" H 5450 3650 50  0001 C CNN
 	1    5450 3650
@@
 	8900 2850 9350 2850
 Wire Wire Line
-	9850 2850 9850 3000
-Wire Wire Line
 	9350 2850 9350 3000
 Connection ~ 9350 2850
 Wire Wire Line
 	9350 2850 9850 2850
-Wire Wire Line
-	9850 4050 9850 3300
 Wire Wire Line
 	8500 3250 8500 4050
@@
 	6250 6650 6250 6450
 Connection ~ 6250 6450
-Wire Wire Line
-	4850 6550 7650 6550
-Wire Wire Line
-	7650 6550 7650 3050
-Connection ~ 7650 3050
 $Comp
 L power:PWR_FLAG #FLG02
@@
 	4600 4050 5450 4050
 Connection ~ 6250 4050
+Wire Wire Line
+	9850 2850 9850 3000
+Wire Wire Line
+	9850 3300 9850 4050
+Wire Wire Line
+	9850 2850 10450 2850
+Wire Wire Line
+	10450 2850 10450 6550
+Wire Wire Line
+	4850 6550 10450 6550
+Connection ~ 9850 2850
 $EndSCHEMATC
