File: hardware/afe/THS5641board/THS5641board/THS5641board.kicad_pcb (KiCad board)
At the start: 2 copper layers, 37 x 53 mm, 24 parts, among them J1 Conn_01x03_Male, J2 Conn_01x03_Male, J3 Conn_02x04_Odd_Even, J4 Conn_01x20_Female, U1 THS5641

Commit message: first THS5641board.kicad_pcb revision
Parts:
- removed D1: LED, LED_SMD:LED_1206_3216Metric
- removed R1: 10 kOhm, Resistor_SMD:R_1206_3216Metric
- added C7: 0.1uF, Capacitor_SMD:C_0805_2012Metric, F.Cu at (79.3, 27.9)
- moved D3 4.65 mm to (80.0, 36.2)
- moved D4 4.65 mm to (80.0, 33.8)
- moved D5 4.65 mm to (80.0, 31.0)
- moved R4 4.65 mm to (87.6, 33.7)
- moved D2 4.65 mm to (79.9, 38.7)
- moved R2 4.65 mm to (87.6, 38.7)
- moved R5 4.65 mm to (87.6, 30.9)
- moved R3 4.65 mm to (87.7, 36.2)
Connections:
- J4 pad 1: Net-(J4-Pad1) -> GND
- J4 pad 10: Net-(J4-Pad10) -> GND
- J4 pad 13: Net-(D1-Pad2) -> GND
- J4 pad 14: Net-(D2-Pad2) -> Net-(J4-Pad14)
- J4 pad 15: Net-(D3-Pad2) -> GND
- J4 pad 16: Net-(D4-Pad2) -> Net-(D2-Pad2)
- J4 pad 17: Net-(D5-Pad2) -> Net-(D3-Pad2)
- J4 pad 18: Net-(J4-Pad18) -> Net-(D4-Pad2)
- J4 pad 19: Net-(J4-Pad19) -> Net-(D5-Pad2)
- J4 pad 20: Net-(J4-Pad20) -> +3V3
- J4 pad 4: Net-(J4-Pad4) -> GND
- J4 pad 7: Net-(J4-Pad7) -> GND
- U1 pad 1: Net-(J4-Pad10) -> Net-(J4-Pad12)
- U1 pad 2: Net-(J4-Pad9) -> Net-(J4-Pad11)
- U1 pad 28: Net-(J4-Pad12) -> Net-(J4-Pad14)
- U1 pad 3: Net-(J4-Pad8) -> Net-(J4-Pad9)
- U1 pad 4: Net-(J4-Pad7) -> Net-(J4-Pad8)
- U1 pad 7: Net-(J4-Pad4) -> Net-(J4-Pad3)
- U1 pad 8: Net-(J4-Pad3) -> Net-(J4-Pad2)
Routing:
- net +3V3: track 99.4 -> 132.3 mm
- net Net-(J4-Pad14): track 0.00 -> 24.1 mm
- net Net-(J4-Pad2): track 0.00 -> 16.4 mm
- net Net-(J4-Pad11): track 0.00 -> 15.3 mm
- net Net-(J4-Pad4): track 14.0 -> 0.00 mm
- net Net-(J4-Pad10): track 13.3 -> 0.00 mm
- net Net-(J4-Pad7): track 12.9 -> 0.00 mm
- net Net-(J4-Pad12): track 23.4 -> 16.0 mm
- net Net-(D1-Pad1): track 4.81 -> 0.00 mm
- net Net-(D1-Pad2): track 3.40 -> 0.00 mm
- net Net-(D5-Pad2): track 3.66 -> 5.47 mm
- net Net-(D3-Pad2): track 3.49 -> 5.23 mm
- net Net-(D4-Pad2): track 3.79 -> 5.43 mm
- net GND: track 0.00 -> 1.53 mm, vias 122 -> 115
- net Net-(D2-Pad2): track 3.69 -> 4.96 mm
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