File: hardware/afe/THS5641board/THS5641board/THS5641board.sch (KiCad schematic (older format))
At the start: 24 parts, among them J1 Conn_01x03_Male, J2 Conn_01x03_Male, J3 Conn_02x04_Odd_Even, J4 Conn_01x20_Female, U1 THS5641

Commit message: first THS5641board.kicad_pcb revision
Parts:
- removed D1: LED, LED_SMD:LED_1206_3216Metric, symbol Device:LED
- removed R1: 10 kOhm, Resistor_SMD:R_1206_3216Metric, symbol Device:R
- added C7: 0.1uF, Capacitor_SMD:C_0805_2012Metric, symbol Device:C
Connections:
- net +3V3: now also J4.20 (Pin_20), C7.1
- net GND: now also J4.1 (Pin_1), J4.10 (Pin_10), J4.13 (Pin_13), J4.15 (Pin_15), J4.4 (Pin_4), J4.7 (Pin_7), C7.2
- net at U1.1 (D7): now also J4.12 (Pin_12); no longer J4.10 (Pin_10)
- net at J4.11 (Pin_11): now also U1.2 (D6)
- net at U1.28 (CLK): now also J4.14 (Pin_14); no longer J4.12 (Pin_12)
- net at D2.2 (A): now also J4.16 (Pin_16); no longer J4.14 (Pin_14)
- net at D3.2 (A): now also J4.17 (Pin_17); no longer J4.15 (Pin_15)
- net at D4.2 (A): now also J4.18 (Pin_18); no longer J4.16 (Pin_16)
- net at D5.2 (A): now also J4.19 (Pin_19); no longer J4.17 (Pin_17)
- net at J4.2 (Pin_2): now also U1.8 (D0)
- net at J4.3 (Pin_3): now also U1.7 (D1); no longer U1.8 (D0)
- net at U1.4 (D4): now also J4.8 (Pin_8); no longer J4.7 (Pin_7)
- net at U1.3 (D5): now also J4.9 (Pin_9); no longer J4.8 (Pin_8)
- no-connect marks 12 -> 6
Changed lines of the file:
@@
 	1    0    0    -1
 $EndComp
-Wire Wire Line
-	6150 2400 7200 2400
-Wire Wire Line
-	6150 2500 7200 2500
-Wire Wire Line
-	6150 2600 7200 2600
-Wire Wire Line
-	6150 2700 7200 2700
-Wire Wire Line
-	6150 2800 7200 2800
-Wire Wire Line
-	6150 2900 7200 2900
-Wire Wire Line
-	6150 3000 7200 3000
-Wire Wire Line
-	6150 3100 7200 3100
 $Comp
 L Connector_Generic:Conn_02x04_Odd_Even J3
@@
 Wire Wire Line
 	3500 1900 3500 1800
-NoConn ~ 7200 3200
-NoConn ~ 7200 4100
-NoConn ~ 7200 4000
 $Comp
 L Connector:Conn_01x03_Male J1
@@
 Wire Wire Line
 	4050 3300 3250 3300
-NoConn ~ 7200 2200
-NoConn ~ 7200 2300
-$Comp
-L Device:LED D1
-U 1 1 5DF85C3A
-P 5900 4550
-F 0 "D1" V 5939 4433 50  0000 R CNN
-F 1 "LED" V 5848 4433 50  0000 R CNN
-F 2 "LED_SMD:LED_1206_3216Metric" H 5900 4550 50  0001 C CNN
-F 3 "~" H 5900 4550 50  0001 C CNN
-	1    5900 4550
-	0    -1   -1   0
-$EndComp
 $Comp
 L Device:LED D2
@@
 $EndComp
 $Comp
-L Device:R R1
-U 1 1 5DF8EF38
-P 5900 5000
-F 0 "R1" H 5970 5046 50  0000 L CNN
-F 1 "10 kOhm" H 5970 4955 50  0000 L CNN
-F 2 "Resistor_SMD:R_1206_3216Metric" V 5830 5000 50  0001 C CNN
-F 3 "~" H 5900 5000 50  0001 C CNN
-	1    5900 5000
-	1    0    0    -1
-$EndComp
-$Comp
 L Device:R R2
 U 1 1 5DF9048D
@@
 $EndComp
 Wire Wire Line
-	5900 5150 5900 5300
-Wire Wire Line
-	5900 5300 6200 5300
-Wire Wire Line
 	6350 5300 6350 5400
 Wire Wire Line
@@
 Wire Wire Line
 	6200 5150 6200 5300
-Connection ~ 6200 5300
 Wire Wire Line
 	6200 5300 6350 5300
 Wire Wire Line
-	5900 4700 5900 4850
-Wire Wire Line
 	6200 4850 6200 4700
 Wire Wire Line
@@
 	6850 4700 6850 4850
 Wire Wire Line
-	7200 3400 6500 3400
-Wire Wire Line
-	6500 3400 6500 3900
-Wire Wire Line
-	6500 3900 5900 3900
-Wire Wire Line
-	5900 3900 5900 4400
-Wire Wire Line
 	6200 4400 6200 4000
 Wire Wire Line
 	6200 4000 6600 4000
 Wire Wire Line
-	6600 4000 6600 3500
-Wire Wire Line
-	6600 3500 7200 3500
-Wire Wire Line
-	7200 3600 6650 3600
-Wire Wire Line
-	6650 3600 6650 4050
+	6600 4000 6600 3700
 Wire Wire Line
 	6650 4050 6450 4050
@@
 	6650 4150 6750 4150
 Wire Wire Line
-	6750 4150 6750 3700
-Wire Wire Line
-	6750 3700 7200 3700
-Wire Wire Line
-	7200 3800 6800 3800
-Wire Wire Line
-	6800 3800 6800 4400
+	6750 4150 6750 3900
 Wire Wire Line
 	6800 4400 6850 4400
-NoConn ~ 7200 3900
 $Comp
 L kilib:THS5641 U1
@@
 	4950 3100 4800 3100
 Wire Wire Line
-	4800 3100 4800 3300
-Wire Wire Line
-	4800 3300 7200 3300
-Wire Wire Line
 	3700 2400 4950 2400
 Wire Wire Line
@@
 NoConn ~ 6150 2200
 NoConn ~ 6150 2300
+$Comp
+L power:+3V3 #PWR06
+U 1 1 5EB8A933
+P 5600 3850
+F 0 "#PWR06" H 5600 3700 50  0001 C CNN
+F 1 "+3V3" H 5615 4023 50  0000 C CNN
+F 2 "" H 5600 3850 50  0001 C CNN
+F 3 "" H 5600 3850 50  0001 C CNN
+	1    5600 3850
+	1    0    0    -1
+$EndComp
+Wire Wire Line
+	5650 3850 5600 3850
+Wire Wire Line
+	5650 3850 5650 4100
+Wire Wire Line
+	5650 4100 7200 4100
+$Comp
+L Device:C C7
+U 1 1 5EB9F2D8
+P 7500 1400
+F 0 "C7" H 7615 1446 50  0000 L CNN
+F 1 "0.1uF" H 7615 1355 50  0000 L CNN
+F 2 "Capacitor_SMD:C_0805_2012Metric" H 7538 1250 50  0001 C CNN
+F 3 "~" H 7500 1400 50  0001 C CNN
+	1    7500 1400
+	1    0    0    -1
+$EndComp
+Wire Wire Line
+	7500 1050 7500 1250
+Wire Wire Line
+	7050 1050 7500 1050
+Wire Wire Line
+	7500 1700 7500 1550
+Wire Wire Line
+	7050 1700 7500 1700
+Wire Wire Line
+	6800 4000 7200 4000
+Wire Wire Line
+	6800 4000 6800 4400
+Wire Wire Line
+	6750 3900 7200 3900
+Wire Wire Line
+	6650 3800 7200 3800
+Wire Wire Line
+	6650 3800 6650 4050
+Wire Wire Line
+	6600 3700 7200 3700
+$Comp
+L power:GND #PWR010
+U 1 1 5EBD2FE3
+P 6050 5650
+F 0 "#PWR010" H 6050 5400 50  0001 C CNN
+F 1 "GND" H 6055 5477 50  0000 C CNN
+F 2 "" H 6050 5650 50  0001 C CNN
+F 3 "" H 6050 5650 50  0001 C CNN
+	1    6050 5650
+	1    0    0    -1
+$EndComp
+Wire Wire Line
+	7200 3600 6400 3600
+Wire Wire Line
+	6050 3600 6050 5650
+Wire Wire Line
+	7200 3500 4800 3500
+Wire Wire Line
+	4800 3100 4800 3500
+Wire Wire Line
+	7200 3400 6400 3400
+Wire Wire Line
+	6400 3400 6400 3600
+Connection ~ 6400 3600
+Wire Wire Line
+	6400 3600 6050 3600
+Wire Wire Line
+	6150 3100 6250 3100
+Wire Wire Line
+	6250 3100 6250 3300
+Wire Wire Line
+	6250 3300 7200 3300
+Wire Wire Line
+	6150 3000 6350 3000
+Wire Wire Line
+	6350 3000 6350 3200
+Wire Wire Line
+	6350 3200 7200 3200
+Wire Wire Line
+	6400 3400 6400 3100
+Wire Wire Line
+	6400 3100 7200 3100
+Connection ~ 6400 3400
+Wire Wire Line
+	6400 3100 6400 2800
+Wire Wire Line
+	6400 2800 7200 2800
+Connection ~ 6400 3100
+Wire Wire Line
+	6400 2800 6400 2500
+Wire Wire Line
+	6400 2200 7200 2200
+Connection ~ 6400 2800
+Wire Wire Line
+	7200 2500 6400 2500
+Connection ~ 6400 2500
+Wire Wire Line
+	6400 2500 6400 2200
+Wire Wire Line
+	6150 2900 6200 2900
+Wire Wire Line
+	6200 2900 6200 2950
+Wire Wire Line
+	6200 2950 6500 2950
+Wire Wire Line
+	6500 2950 6500 3000
+Wire Wire Line
+	6500 3000 7200 3000
+Wire Wire Line
+	6150 2800 6300 2800
+Wire Wire Line
+	6300 2800 6300 2850
+Wire Wire Line
+	6300 2850 6550 2850
+Wire Wire Line
+	6550 2850 6550 2900
+Wire Wire Line
+	6550 2900 7200 2900
+Wire Wire Line
+	6150 2700 7200 2700
+Wire Wire Line
+	6150 2600 7200 2600
+Wire Wire Line
+	6300 2400 6300 2300
+Wire Wire Line
+	6300 2300 7200 2300
+Wire Wire Line
+	6150 2400 6300 2400
+Wire Wire Line
+	6150 2500 6350 2500
+Wire Wire Line
+	6350 2500 6350 2400
+Wire Wire Line
+	6350 2400 7200 2400
 $EndSCHEMATC
