File: hardware/afe/ADC08100board/ADC08100board/ADC08100board.kicad_pcb (KiCad board)
At the start: 2 copper layers, 37 x 53 mm, 21 parts, among them J1 Conn_01x03_Male, J3 Conn_02x04_Odd_Even, J4 Conn_01x20_Female, U1 ADC08060

Commit message: first ADC08100board.kicad_pcb revision
Parts:
- removed D1: LED, LED_SMD:LED_1206_3216Metric
- removed R1: 10 kOhm, Resistor_SMD:R_1206_3216Metric
- added C6: 0.1uF, Capacitor_SMD:C_0805_2012Metric, F.Cu at (78.8, 28.2)
- moved D2 4.01 mm to (80.3, 39.5)
- moved D3 4.01 mm to (80.3, 37.0)
- moved D4 4.01 mm to (80.3, 34.6)
- moved D5 4.01 mm to (80.4, 31.9)
- moved R2 4.01 mm to (88.0, 39.5)
- moved R4 4.01 mm to (87.9, 34.5)
- moved R5 4.01 mm to (87.9, 31.8)
- moved R3 4.01 mm to (88.0, 37.1)
Connections:
- J4 pad 1: Net-(J4-Pad1) -> GND
- J4 pad 10: Net-(J4-Pad10) -> GND
- J4 pad 13: Net-(D1-Pad2) -> GND
- J4 pad 14: Net-(D2-Pad2) -> Net-(J4-Pad14)
- J4 pad 15: Net-(D3-Pad2) -> GND
- J4 pad 16: Net-(D4-Pad2) -> Net-(D2-Pad2)
- J4 pad 17: Net-(D5-Pad2) -> Net-(D3-Pad2)
- J4 pad 18: Net-(J4-Pad18) -> Net-(D4-Pad2)
- J4 pad 19: Net-(J4-Pad19) -> Net-(D5-Pad2)
- J4 pad 20: Net-(J4-Pad20) -> +3V3
- J4 pad 4: Net-(J4-Pad4) -> GND
- J4 pad 7: Net-(J4-Pad7) -> GND
- U1 pad 13: Net-(J4-Pad3) -> Net-(J4-Pad2)
- U1 pad 14: Net-(J4-Pad4) -> Net-(J4-Pad3)
- U1 pad 19: Net-(J4-Pad7) -> Net-(J4-Pad8)
- U1 pad 20: Net-(J4-Pad8) -> Net-(J4-Pad9)
- U1 pad 21: Net-(J4-Pad9) -> Net-(J4-Pad11)
- U1 pad 22: Net-(J4-Pad10) -> Net-(J4-Pad12)
- U1 pad 24: Net-(J4-Pad12) -> Net-(J4-Pad14)
Routing:
- net +3V3: track 89.2 -> 128.4 mm
- net Net-(J4-Pad2): track 0.00 -> 16.3 mm
- net Net-(J4-Pad14): track 0.00 -> 15.9 mm
- net Net-(J4-Pad4): track 12.5 -> 0.00 mm
- net Net-(J4-Pad11): track 0.00 -> 10.8 mm
- net Net-(J4-Pad7): track 10.4 -> 0.00 mm
- net Net-(J4-Pad10): track 9.37 -> 0.00 mm
- net Net-(D1-Pad1): track 4.81 -> 0.00 mm
- net Net-(D1-Pad2): track 3.40 -> 0.00 mm
- net Net-(D3-Pad2): track 3.49 -> 6.27 mm
- net Net-(D5-Pad2): track 3.66 -> 5.85 mm
- net Net-(D4-Pad2): track 3.79 -> 5.99 mm
- net Net-(D2-Pad2): track 3.69 -> 5.89 mm
- net GND: track 0.00 -> 1.20 mm, vias 140 -> 184
- net Net-(J4-Pad3): track 13.7 -> 14.7 mm
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Other:
- net class Default: clearance 0.2 -> 0.15; trace_width 0.25 -> 0.15; via_dia 0.8 -> 0.5; via_drill 0.4 -> 0.25
- rule trace_clearance: 0.2 -> 0.15
- rule trace_min: 0.2 -> 0.15
- rule via_min_drill: 0.3 -> 0.25
- rule via_min_size: 0.4 -> 0.5
