File: hardware/power/power-12v/power3X/power3X.kicad_pcb (KiCad board)
At the start: 2 copper layers, 37 x 53 mm, 17 parts, among them J1 Conn_01x20_Male, U1 TPS560200, U2 MAX40200AUK

Commit message: started Power 12V board skeleton
Parts:
- removed BT1, BT2, BT3, BT4: Battery_Cell, kifootp:CR2032
- added J2: Conn_01x02_Male, Connector_PinHeader_2.54mm:PinHeader_1x02_P2.54mm_Vertical, F.Cu at (91.1, 32.0)
Routing:
- net Net-(C1-Pad1): track 58.6 -> 63.3 mm
- net Net-(BT3-Pad2): track 58.6 -> 63.1 mm
- net Net-(BT1-Pad2): track 63.3 -> 67.2 mm
- net Net-(BT2-Pad2): track 67.9 -> 70.8 mm
