File: hardware/perif/electrolyzer/electrolyzer/pwm_ctl1.sch (KiCad schematic (older format))
At the start: 0 parts

Commit message: Started Electrolyzer board: sense
Parts:
- added J?: Conn_01x20_Female, symbol Connector:Conn_01x20_Female
Changed lines of the file:
@@
 Comment4 ""
 $EndDescr
+$Comp
+L Connector:Conn_01x20_Female J?
+U 1 1 5F21D68C
+P 3150 2850
+F 0 "J?" H 3042 1625 50  0000 C CNN
+F 1 "Conn_01x20_Female" H 3042 1716 50  0000 C CNN
+F 2 "" H 3150 2850 50  0001 C CNN
+F 3 "~" H 3150 2850 50  0001 C CNN
+	1    3150 2850
+	-1   0    0    1
+$EndComp
 $EndSCHEMATC
